File: eagle/tempeh_Hat.sch (EAGLE design)
At the start: 8 parts, among them K1 PIN20X2

Commit message: adding pcb v1
Connections:
- net +3V3: no longer K1.17
- net GND: no longer K1.6, K1.9
Changed lines of the file:
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@@
 <net name="GND" class="0">
 <segment>
-<pinref part="K1" gate="G$1" pin="9"/>
 <pinref part="GND3" gate="1" pin="GND"/>
-<wire x1="43.18" y1="165.1" x2="40.64" y2="165.1" width="0.1524" layer="91"/>
-<wire x1="40.64" y1="165.1" x2="40.64" y2="144.78" width="0.1524" layer="91"/>
 <pinref part="K1" gate="G$1" pin="25"/>
 <wire x1="40.64" y1="144.78" x2="40.64" y2="127" width="0.1524" layer="91"/>
@@
 <pinref part="K1" gate="G$1" pin="39"/>
 <wire x1="43.18" y1="127" x2="40.64" y2="127" width="0.1524" layer="91"/>
-<junction x="40.64" y="144.78"/>
 <junction x="40.64" y="127"/>
 </segment>
 <segment>
-<pinref part="K1" gate="G$1" pin="6"/>
 <pinref part="GND10" gate="1" pin="GND"/>
-<wire x1="58.42" y1="170.18" x2="60.96" y2="170.18" width="0.1524" layer="91"/>
-<wire x1="60.96" y1="170.18" x2="60.96" y2="160.02" width="0.1524" layer="91"/>
 <pinref part="K1" gate="G$1" pin="14"/>
 <wire x1="60.96" y1="160.02" x2="60.96" y2="152.4" width="0.1524" layer="91"/>
@@
 <pinref part="K1" gate="G$1" pin="34"/>
 <wire x1="58.42" y1="134.62" x2="60.96" y2="134.62" width="0.1524" layer="91"/>
-<junction x="60.96" y="160.02"/>
 <junction x="60.96" y="152.4"/>
 <junction x="60.96" y="139.7"/>
@@
 <wire x1="43.18" y1="175.26" x2="38.1" y2="175.26" width="0.1524" layer="91"/>
 <wire x1="38.1" y1="175.26" x2="38.1" y2="180.34" width="0.1524" layer="91"/>
-<pinref part="K1" gate="G$1" pin="17"/>
-<wire x1="43.18" y1="154.94" x2="38.1" y2="154.94" width="0.1524" layer="91"/>
-<wire x1="38.1" y1="154.94" x2="38.1" y2="175.26" width="0.1524" layer="91"/>
-<junction x="38.1" y="175.26"/>
 </segment>
 <segment>
