File: eagle/tempeh_NoHat.brd (EAGLE design)
At the start: 7 x 7.1 mm, 7 parts, among them K1 PIN20X2

Commit message: new version of pcb board
Routing:
- net GND: track 76.8 -> 78.4 mm
Changed lines of the file:
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@@
 <classes>
 <class number="0" name="default" width="0.3048" drill="0.508">
-<clearance class="0" value="0.254"/>
+<clearance class="0" value="0.0254"/>
 </class>
 </classes>
@@
 <wire x1="9.46" y1="28.46" x2="19" y2="38" width="1.016" layer="16"/>
 <wire x1="19" y1="38" x2="19" y2="41" width="1.016" layer="16"/>
-<wire x1="19" y1="41" x2="21" y2="43" width="1.016" layer="16"/>
-<wire x1="54.4" y1="43" x2="56.63" y2="45.23" width="1.016" layer="16"/>
-<wire x1="21" y1="43" x2="54.4" y2="43" width="1.016" layer="16"/>
+<wire x1="19" y1="41" x2="20.508" y2="42.508" width="1.016" layer="16"/>
+<wire x1="56.63" y1="42.508" x2="56.63" y2="45.23" width="1.016" layer="16"/>
+<wire x1="20.508" y1="42.508" x2="56.63" y2="42.508" width="1.016" layer="16"/>
 </signal>
 <signal name="+3V3">
@@
 <contactref element="K1" pad="2"/>
 <contactref element="RELAY" pad="2"/>
-<wire x1="2" y1="44" x2="5" y2="44" width="1.016" layer="16"/>
-<wire x1="5" y1="44" x2="5.5" y2="44.5" width="1.016" layer="16"/>
-<wire x1="5.5" y1="44.5" x2="6" y2="45" width="1.016" layer="16"/>
-<wire x1="6" y1="45" x2="6" y2="46" width="1.016" layer="16"/>
-<wire x1="6" y1="46" x2="7.77" y2="47.77" width="1.016" layer="16"/>
-<wire x1="7.77" y1="47.77" x2="8.37" y2="47.77" width="1.016" layer="16"/>
+<wire x1="2" y1="44" x2="5" y2="44" width="0.8128" layer="16"/>
+<wire x1="5" y1="44" x2="6" y2="45" width="0.6096" layer="16"/>
+<wire x1="6" y1="45" x2="6" y2="46" width="0.6096" layer="16"/>
+<wire x1="6" y1="46" x2="7.77" y2="47.77" width="0.6096" layer="16"/>
+<wire x1="7.77" y1="47.77" x2="8.37" y2="47.77" width="0.8128" layer="16"/>
 </signal>
 <signal name="N$2">
